File: SPI_Protocol_Connector.kicad_sch (KiCad schematic)
At the start: 8 parts, among them J5 Conn_01x03_Pin, J7 Conn_01x06_Pin, U4 TXU0104PWR, U5 TXU0104PWR

Commit message: most routing done
Connections:
- net V_2nd is gone; now on net V_SEL: J5.2 (Pin_2)
Changed lines of the file:
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@@
 		)
 	)
-	(label "V_2nd"
+	(label "V_SEL"
 		(at 40.64 163.83 180)
 		(effects
