File: MMS3_hat_protocol.kicad_sch (KiCad schematic)
At the start: 49 parts, among them J10 Conn_01x02_Pin, J3 Conn_01x02_Pin, J4 Conn_01x04_Pin, J6 Conn_01x04_Pin, J9 Conn_01x04_Pin, U13 TCA9535PWR_C130204, U3 AMS1117, U9 PCA9306DCUR

Commit message: most routing done
Parts:
- removed PN1: (no value), PCM_JLCPCB:Part_Num_JLCPCB, symbol PCM_JLCPCB-Manufacturing:Part Number, PCM_JLCPCB, 0.8x0.15mm
- added D19, D20, D21, D22, D23, D24, D25, D26: Red, PCM_JLCPCB:D_0603, symbol PCM_JLCPCB-Diodes:LED,0603,Red
- added R45, R46, R47, R48, R49, R50, R51, R52: 330Ω, PCM_JLCPCB:R_0402, symbol PCM_JLCPCB-Resistors:0402,330Ω
Connections:
- net +5V: no longer C22.1
- net GND: now also D19.1, D20.1, D21.1, D22.1, D23.1, D24.1, D25.1, D26.1
- net P03: now also R45.1
- net P04: now also R46.1
- net P11: now also R47.1
- net P12: now also R48.1
- net P14: now also R51.1
- net P15: now also R52.1
- net P16: now also R49.1
- net P17: now also R50.1
- net Vref2: now reaches R7.1, U9.7 (VREF2), U9.8 (EN)
- net Vref2: now also C22.1
- new net: D26.2, R52.2
- new net: D19.2, R45.2
- new net: D25.2, R51.2
- new net: D23.2, R49.2
- new net: D24.2, R50.2
- new net: D22.2, R48.2
- new net: D21.2, R47.2
- new net: D20.2, R46.2
Other:
- moved on the sheet: D10, D15, D16, D17, D18, D8, D9, J10, J3, J9, R10, R11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
