File: UART_Protocol_Connector.kicad_sch (KiCad schematic)
At the start: 19 parts, among them J11 Conn_01x04_Pin, J8 Conn_01x03_Pin, U11 TXU0104PWR, U6 MAX13487EESA, U8 TXU0104PWR

Commit message: most routing done
Parts:
- removed D11, D13: Red, PCM_JLCPCB:D_0603, symbol PCM_JLCPCB-Diodes:LED,0603,Red
- removed R29, R31: 330Ω, PCM_JLCPCB:R_0402, symbol PCM_JLCPCB-Resistors:0402,330Ω
- removed R33, R35: 10kΩ, PCM_JLCPCB:R_0402, symbol PCM_JLCPCB-Resistors:0402,10kΩ
Connections:
- net V_2nd is gone; now on net V_SEL: J8.2 (Pin_2)
