File: MMS3_hat_protocol.kicad_pcb (KiCad board)
At the start: 2 copper layers, 100 x 50 mm, 80 parts, among them J1 Chainbus in, J11 Conn_01x04_Pin, J12 Conn_01x04_Pin, J13 Conn_01x04_Pin, J14 Conn_01x03_Pin, J15 Conn_01x04_Pin, J2 Chainbus Out, J4 Conn_01x04_Pin, J5 Conn_01x03_Pin, J6 Conn_01x04_Pin, J7 Conn_01x06_Pin, J8 Conn_01x03_Pin, J9 Conn_01x04_Pin, U1 SN74CB3Q3384APW, U10 TXU0104PWR, U11 TXU0104PWR, U12 TXU0104PWR, U2 M24C64, U3 AMS1117, U4 TXU0104PWR, U5 TXU0104PWR, U7 MAX3483ESA+T, U8 TXU0104PWR, U9 PCA9306DCUR

Commit message: most routing done
Parts:
- removed J12, J13: Conn_01x04_Pin, Connector_JST:JST_XH_S4B-XH-A_1x04_P2.50mm_Horizontal
- removed PN1: ~, PCM_JLCPCB:Part_Num_JLCPCB
- removed U7: MAX3483ESA+T, MAX3483ESA:PG-DSO-8_L5.0-W4.0-P1.27-LS6.0-BL
- added C12: 100nF, PCM_JLCPCB:C_0603, F.Cu at (125.8, 115.4)
- added C14: 100nF, PCM_JLCPCB:C_0603, F.Cu at (143.9, 115.4)
- added D15: Red, PCM_JLCPCB:D_0603, F.Cu at (85.7, 104.8)
- added D16: Red, PCM_JLCPCB:D_0603, F.Cu at (85.7, 106.7)
- added D17: Red, PCM_JLCPCB:D_0603, F.Cu at (85.7, 123.5)
- added D18: Red, PCM_JLCPCB:D_0603, F.Cu at (85.7, 101.1)
- added D19: Red, PCM_JLCPCB:D_0603, F.Cu at (85.7, 103.0)
- added D20: Red, PCM_JLCPCB:D_0603, F.Cu at (85.7, 95.5)
- added D21: Red, PCM_JLCPCB:D_0603, F.Cu at (85.7, 121.6)
- added D22: Red, PCM_JLCPCB:D_0603, F.Cu at (85.8, 119.7)
- added D23: Red, PCM_JLCPCB:D_0603, F.Cu at (85.7, 112.3)
- added D24: Red, PCM_JLCPCB:D_0603, F.Cu at (85.7, 110.4)
- added D25: Red, PCM_JLCPCB:D_0603, F.Cu at (85.7, 116.0)
- added D26: Red, PCM_JLCPCB:D_0603, F.Cu at (85.7, 114.2)
- added J10: Conn_01x02_Pin, Connector_PinSocket_2.54mm:PinSocket_1x02_P2.54mm_Vertical, F.Cu at (150.9, 129.6)
- added J3: Conn_01x02_Pin, Connector_PinSocket_2.54mm:PinSocket_1x02_P2.54mm_Vertical, F.Cu at (132.7, 129.4)
- added R23: 510Ω, PCM_JLCPCB:R_0603, F.Cu at (119.6, 118.2)
- added R24: 510Ω, PCM_JLCPCB:R_0603, F.Cu at (137.7, 118.0)
- added R25: 120Ω, PCM_JLCPCB:R_0603, F.Cu at (122.4, 118.2)
- added R26: 510Ω, PCM_JLCPCB:R_0603, F.Cu at (125.2, 118.2)
- added R27: 510Ω, PCM_JLCPCB:R_0603, F.Cu at (143.0, 118.0)
- added R28: 120Ω, PCM_JLCPCB:R_0603, F.Cu at (140.4, 118.0)
- added R37: 330Ω, PCM_JLCPCB:R_0402, F.Cu at (88.3, 104.8)
- added R38: 10kΩ, PCM_JLCPCB:R_0402, F.Cu at (66.9, 113.2)
- added R39: 330Ω, PCM_JLCPCB:R_0402, F.Cu at (88.3, 106.7)
- added R40: 10kΩ, PCM_JLCPCB:R_0402, F.Cu at (66.9, 115.1)
- added R41: 330Ω, PCM_JLCPCB:R_0402, F.Cu at (88.3, 123.5)
- added R42: 10kΩ, PCM_JLCPCB:R_0402, F.Cu at (66.9, 116.9)
- added R43: 330Ω, PCM_JLCPCB:R_0402, F.Cu at (88.3, 101.1)
- added R44: 10kΩ, PCM_JLCPCB:R_0402, F.Cu at (66.9, 118.8)
- added R45: 330Ω, PCM_JLCPCB:R_0402, F.Cu at (88.3, 103.0)
- added R46: 330Ω, PCM_JLCPCB:R_0402, F.Cu at (88.3, 95.5)
- added R47: 330Ω, PCM_JLCPCB:R_0402, F.Cu at (88.3, 121.6)
- added R48: 330Ω, PCM_JLCPCB:R_0402, F.Cu at (88.4, 119.7)
- added R49: 330Ω, PCM_JLCPCB:R_0402, F.Cu at (88.3, 112.3)
- added R50: 330Ω, PCM_JLCPCB:R_0402, F.Cu at (88.3, 110.4)
- added R51: 330Ω, PCM_JLCPCB:R_0402, F.Cu at (88.3, 116.0)
- added R52: 330Ω, PCM_JLCPCB:R_0402, F.Cu at (88.3, 114.2)
- added U13: TCA9535PWR_C130204, TCA9535PWR:TSSOP-24_L7.8-W4.4-P0.65-LS6.4-BL, F.Cu at (107.6, 109.4)
- added U15: MAX13487EESA, MAX13487EESA:SOIC-8_L4.9-W3.9-P1.27-LS6.0-BL, F.Cu at (140.5, 113.6)
- added U6: MAX13487EESA, MAX13487EESA:SOIC-8_L4.9-W3.9-P1.27-LS6.0-BL, F.Cu at (122.4, 113.6)
- J14, J5, J8: footprint Connector_PinSocket_2.54mm:PinSocket_1x03_P2.54mm_Vertical -> Connector_PinSocket_2.54mm:PinSocket_1x03_P2.54mm_Horizontal
- J9: footprint Connector_JST:JST_XH_S4B-XH-A_1x04_P2.50mm_Horizontal -> Connector_PinSocket_2.54mm:PinSocket_1x04_P2.54mm_Vertical
- moved R15 164.8 mm to (62.0, 115.1)
- moved R16 164.8 mm to (62.0, 116.9)
- moved R17 164.8 mm to (62.0, 118.8)
- moved R18 164.8 mm to (62.0, 120.6)
- moved R19 164.8 mm to (62.0, 122.5)
- moved R20 164.8 mm to (62.0, 124.3)
- moved R3 164.8 mm to (62.0, 111.4)
- moved R4 164.8 mm to (62.0, 113.2)
- moved R2 157.0 mm to (62.0, 109.5), turned to 0 degrees
- moved R10 152.4 mm to (66.9, 109.5)
- moved R11 152.4 mm to (66.9, 111.4)
- moved C2 146.9 mm to (96.0, 127.0), turned to -90 degrees
- moved R14 131.0 mm to (88.3, 117.9), turned to 180 degrees
- moved R13 130.7 mm to (88.3, 99.2), turned to 180 degrees
- moved R12 130.7 mm to (88.3, 108.6), turned to 180 degrees
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Connections:
- net /P01 renamed /UART 1/Bonus_IN_1_3V3
- net /P07 renamed /UART 2/Bonus_IN_1_3V3
- net /UART 1/RX_SEL renamed /UART 1/RS485_A
- net /UART 1/TX_SEL renamed /UART 1/RS485_B
- net /UART 2/RX_SEL renamed /UART 2/RS485_A
- net /UART 2/TX_SEL renamed /UART 2/RS485_B
- C22 pad 1: +5V -> /Vref2
- D6 pad 1: GND -> Net-(D6-Pad1)
- D6 pad 2: Net-(D6-Pad2) -> +3V3
- J14 pad 2: /UART 2/V_2nd -> /UART 2/V_SEL
- J5 pad 2: /SPI 1/V_2nd -> /SPI 1/V_SEL
- J8 pad 2: /UART 1/V_2nd -> /UART 1/V_SEL
- R11 pad 2: +3V3 -> GND
- R21 pad 2: Net-(D6-Pad2) -> Net-(D6-Pad1)
- R6 pad 2: +3V3 -> GND
- R7 pad 1: Net-(U9-EN) -> /Vref2
- U10 pad 10: /UART 2/Bonus_OUT_3_SEL -> unconnected-(U10-B4Y-Pad10)
- U10 pad 5: /P10 -> unconnected-(U10-A4-Pad5)
- U11 pad 10: /UART 1/Bonus_OUT_3_SEL -> unconnected-(U11-B4Y-Pad10)
- U11 pad 5: /P02 -> unconnected-(U11-A4-Pad5)
- U12 pad 10: /UART 2/Bonus_IN_3_3V3 -> unconnected-(U12-B4Y-Pad10)
- U12 pad 5: /UART 2/Bonus_IN_3_SEL -> unconnected-(U12-A4-Pad5)
- U8 pad 10: /UART 1/Bonus_IN_3_3V3 -> unconnected-(U8-B4Y-Pad10)
- U8 pad 5: /UART 1/Bonus_IN_3_SEL -> unconnected-(U8-A4-Pad5)
- U9 pad 7: Net-(U9-EN) -> /Vref2
- U9 pad 8: Net-(U9-EN) -> /Vref2
Routing:
- net +3V3: track 0.00 -> 363.6 mm, vias 0 -> 10
- net +5V: track 0.00 -> 207.4 mm, vias 4 -> 11
- net /P16: track 0.00 -> 147.2 mm, vias 0 -> 4
- net /P15: track 0.00 -> 131.0 mm, vias 0 -> 2
- net /P14: track 0.00 -> 127.4 mm, vias 0 -> 2
- net /P13: track 0.00 -> 120.3 mm, vias 0 -> 4
- net /P17: track 0.00 -> 115.8 mm, vias 0 -> 4
- net /UART 1/V_SEL: track 0.00 -> 111.1 mm, vias 0 -> 4
- net /P12: track 0.00 -> 110.8 mm, vias 0 -> 2
- net /P11: track 0.00 -> 109.3 mm, vias 0 -> 2
- net /UART 2/V_SEL: track 0.00 -> 80.2 mm, vias 0 -> 1
- net /P06: track 0.00 -> 79.2 mm, vias 0 -> 8
- net /Bus_switch/SEL1: track 20.6 -> 90.9 mm, vias 0 -> 9
- net /Chainbus.SDA: track 0.00 -> 70.3 mm, vias 0 -> 4
- net /Chainbus.SCL: track 0.00 -> 69.5 mm, vias 0 -> 4
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Other:
- board text added: "8"
- board text added: "MMS3 HAT Protocol"
- board text added: "SEL"
- board text added: "UART1"
- board text added: "UART2"
- board text added: "expander P05"
- board text added: "rs485_1 rec en"
- board text added: "rs485_1 shutdown"
- board text added: "rs485_2 rec en"
- board text added: "rs485_2 shutdown"
- board text added: "spi OE"
- board text added: "spi bonus I1"
- board text added: "spi bonus I2"
- board text added: "spi bonus I3"
- board text added: "spi bonus O1"
- board text added: "uart1 OE"
- board text added: "uart1 bonus O1"
- board text added: "uart1 bonus O2"
- board text added: "uart2 OE"
- board text added: "uart2 bonus O1"
- board text added: "uart2 bonus O2"
- board text removed: "2"
- board text removed: "Selected"

Commit message: finished routing
Parts:
- moved R18 101.9 mm to (163.9, 121.6), turned to 180 degrees
- moved R3 97.9 mm to (159.5, 120.8), turned to 180 degrees
- moved R4 97.7 mm to (159.5, 119.8)
- moved R20 96.1 mm to (157.9, 117.9)
- moved R2 89.0 mm to (150.8, 115.7)
- moved R16 71.7 mm to (133.1, 107.5), turned to -90 degrees
- moved R17 69.6 mm to (131.1, 110.5), turned to -90 degrees
- moved R10 69.3 mm to (136.1, 113.0)
- moved R44 62.9 mm to (127.5, 102.1)
- moved R11 53.7 mm to (120.0, 119.4)
- moved R38 50.8 mm to (116.7, 103.4)
- moved R15 49.2 mm to (111.1, 118.6), turned to 180 degrees
- moved R40 49.1 mm to (114.9, 104.8), turned to -90 degrees
- moved R42 47.8 mm to (114.7, 116.7), turned to -90 degrees
- moved R19 38.3 mm to (100.2, 125.2)
Routing:
- net +3V3: track 363.6 -> 381.9 mm, vias 10 -> 13
- net GND: track 56.7 -> 71.7 mm, vias 46 -> 263
- net /SPI 1/V_SEL: track 29.4 -> 33.0 mm
- net /Chainbus.SCK: track 30.6 -> 33.9 mm, vias 2 -> 4
- net /Chainbus.TX: track 57.1 -> 59.2 mm, vias 5 -> 6
- net /P10: track 65.1 -> 66.6 mm, vias 4 -> 5
- net /UART 2/V_SEL: track 80.2 -> 78.9 mm
- net /P17: track 115.8 -> 117.0 mm
- net /P07: track 67.7 -> 68.6 mm
- net /Chainbus.CS: track 28.7 -> 29.5 mm, vias 2 -> 3
- net /P16: track 147.2 -> 147.8 mm
- net /P02: track 46.2 -> 46.8 mm
Other:
- board text added: "3"
- board text added: "3V3"
- board text added: "5V"
- board text added: "CS"
- board text added: "GND"
- board text added: "MISO"
- board text added: "MOSI"
- board text added: "RX/A"
- board text added: "Remove when using UART"
- board text added: "SCK"
- board text added: "SCL"
- board text added: "SDA"
- board text added: "TX/B"
- board text added: "Use Jumper to select ouput bus voltage"
- board text added: "VCC"
- board text removed: "8"
